File: micro-d-tes-aaray - ryan_copy/micro-d-tes-aaray.kicad_pcb (KiCad board)
At the start: 4 copper layers, 32 x 60 mm, 46 parts, among them J1 Conn_01x01_Socket, J10 Conn_01x01_Socket, J11 Conn_01x01_Socket, J12 Conn_01x01_Socket, J13 Conn_01x01_Socket, J14 Conn_01x01_Socket, J15 Conn_01x01_Socket, J16 Conn_01x01_Socket, J17 Conn_01x01_Socket, J18 Conn_01x01_Socket, J19 Conn_01x01_Socket, J2 Conn_01x01_Socket, J20 Conn_01x01_Socket, J21 DB25_Plug, J22 Conn_01x01_Socket, J23 Conn_01x01_Socket, J24 Conn_01x01_Socket, J25 Conn_01x01_Socket, J26 Conn_01x01_Socket, J27 Conn_01x01_Socket, J28 Conn_01x01_Socket, J29 Conn_01x01_Socket, J3 Conn_01x01_Socket, J30 Conn_01x01_Socket, J31 Conn_01x01_Socket, J32 Conn_01x01_Socket, J33 Conn_01x01_Socket, J34 Conn_01x01_Socket, J35 Conn_01x01_Socket, J36 Conn_01x01_Socket, J37 Conn_01x01_Socket, J38 Conn_01x01_Socket, J39 Conn_01x01_Socket, J4 Conn_01x01_Socket, J40 Conn_01x01_Socket, J41 Conn_01x01_Socket, J42 DB25_Plug, J5 Conn_01x01_Socket, J6 Conn_01x01_Socket, J7 Conn_01x01_Socket, J8 Conn_01x01_Socket, J9 Conn_01x01_Socket

Commit message: update
Parts:
- added D11: Conn_01x01_Socket, 0_footprint_Library:SolderWirePad_1x01_SMD_0.5x0.5mm, F.Cu at (29.0, 40.8)
- added D12: Conn_01x01_Socket, 0_footprint_Library:SolderWirePad_1x01_SMD_0.5x0.5mm, F.Cu at (31.5, 40.8)
- added D24: Conn_01x01_Socket, 0_footprint_Library:SolderWirePad_1x01_SMD_0.5x0.5mm, F.Cu at (30.2, 40.8)
- added D25: Conn_01x01_Socket, 0_footprint_Library:SolderWirePad_1x01_SMD_0.5x0.5mm, F.Cu at (32.7, 40.8)
- added J11: Conn_01x01_Socket, 0_footprint_Library:SolderWirePad_1x01_SMD_0.5x0.5mm, F.Cu at (6.50, 22.7)
- added J12: Conn_01x01_Socket, 0_footprint_Library:SolderWirePad_1x01_SMD_0.5x0.5mm, F.Cu at (3.97, 22.7)
- added J24: Conn_01x01_Socket, 0_footprint_Library:SolderWirePad_1x01_SMD_0.5x0.5mm, F.Cu at (5.22, 22.7)
- added J25: Conn_01x01_Socket, 0_footprint_Library:SolderWirePad_1x01_SMD_0.5x0.5mm, F.Cu at (2.72, 22.7)
- moved J1 4.18 mm to (31.5, 22.7)
- moved J10 4.18 mm to (9.00, 22.7)
- moved J14 4.18 mm to (30.2, 22.7)
- moved J15 4.18 mm to (27.8, 22.7)
- moved J16 4.18 mm to (25.2, 22.7)
- moved J17 4.18 mm to (22.8, 22.7)
- moved J18 4.18 mm to (20.2, 22.7)
- moved J19 4.18 mm to (17.8, 22.7)
- moved J2 4.18 mm to (29.0, 22.7)
- moved J20 4.18 mm to (15.2, 22.7)
- moved J21 4.18 mm to (12.8, 22.7)
- moved J22 4.18 mm to (10.2, 22.7)
- moved J23 4.18 mm to (7.75, 22.7)
- moved J3 4.18 mm to (26.5, 22.7)
- moved J4 4.18 mm to (24.0, 22.7)
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- renumbered J19 to D1, J1 to D10, J18 to D14, J16 to D15, J14 to D16, J12 to D17, J10 to D18, J8 to D19, J17 to D2, J6 to D20, J4 to D21, J2 to D22, J20 to D23, J15 to D3, J13 to D4, J11 to D5, J9 to D6, J7 to D7, J5 to D8, J3 to D9, H4 to H2, H2 to H3, H3 to H4, J40 to J1, J22 to J10, J42 to J13, J39 to J14, J37 to J15, J35 to J16, J33 to J17, J31 to J18, J29 to J19, J38 to J2, J27 to J20, J25 to J21, J23 to J22, J41 to J23, J21 to J26, J36 to J3, J34 to J4, J32 to J5, J30 to J6, J28 to J7, J26 to J8, J24 to J9
Connections:
- J13 pad 11: unconnected-(J42-Pad11) -> Net-(J11-Pin_1)
- J13 pad 12: unconnected-(J42-Pad12) -> Net-(J12-Pin_1)
- J13 pad 24: unconnected-(J42-P24-Pad24) -> Net-(J13-P24)
- J13 pad 25: unconnected-(J42-P25-Pad25) -> Net-(J13-P25)
- J26 pad 11: unconnected-(J21-Pad11) -> Net-(D11-Pin_1)
- J26 pad 12: unconnected-(J21-Pad12) -> Net-(D12-Pin_1)
- J26 pad 24: unconnected-(J21-P24-Pad24) -> Net-(D24-Pin_1)
- J26 pad 25: unconnected-(J21-P25-Pad25) -> Net-(D25-Pin_1)
Routing:
- net Net-(D4-Pin_1): track 0.00 -> 23.7 mm, vias 0 -> 1
- net Net-(J8-Pin_1): track 0.00 -> 22.4 mm, vias 0 -> 1
- net Net-(D3-Pin_1): track 0.00 -> 21.9 mm, vias 0 -> 1
- net Net-(D16-Pin_1): track 0.00 -> 21.4 mm, vias 0 -> 1
- net Net-(J3-Pin_1): track 0.00 -> 20.8 mm, vias 0 -> 1
- net Net-(D2-Pin_1): track 0.00 -> 20.7 mm, vias 0 -> 1
- net Net-(J7-Pin_1): track 0.00 -> 20.6 mm, vias 0 -> 1
- net Net-(J13-P20): track 0.00 -> 20.5 mm, vias 0 -> 1
- net Net-(D7-Pin_1): track 0.00 -> 20.3 mm, vias 0 -> 1
- net Net-(J13-P21): track 0.00 -> 20.3 mm, vias 0 -> 1
- net Net-(J13-P16): track 0.00 -> 20.2 mm, vias 0 -> 1
- net Net-(D15-Pin_1): track 0.00 -> 20.2 mm, vias 0 -> 1
- net Net-(D20-Pin_1): track 0.00 -> 20.1 mm, vias 0 -> 1
- net Net-(D12-Pin_1): track 0.00 -> 19.8 mm, vias 0 -> 1
- net Net-(J12-Pin_1): track 0.00 -> 19.8 mm, vias 0 -> 1
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Other:
- board size 32 x 60 mm -> 35.5 x 63.5 mm

Commit message: update pcb
Parts:
- removed the J10 at (9.00, 22.7)
- removed the J23 at (7.75, 22.7)
- added D13: Conn_01x01_Socket, 0_footprint_Library:SolderWirePad_1x01_SMD_0.5x2mm_1, F.Cu at (28.0, 38.0)
- added J13: Conn_01x01_Socket, 0_footprint_Library:SolderWirePad_1x01_SMD_0.7x2mm, F.Cu at (7.50, 25.5)
- added J20: Conn_01x01_Socket, 0_footprint_Library:SolderWirePad_1x01_SMD_0.5x2mm_1, F.Cu at (16.3, 25.5)
- added J7: Conn_01x01_Socket, 0_footprint_Library:SolderWirePad_1x01_SMD_0.7x2mm, F.Cu at (17.1, 25.5)
- D1, D10, D11, D12, D14, D15, D16, D17, D19, D2, D20, D21, D22, D24, D25, D4, D5, D6, D7, D9, J1, J11, J12, J2, J3, J4, J5, J6: footprint 0_footprint_Library:SolderWirePad_1x01_SMD_0.5x0.5mm -> 0_footprint_Library:SolderWirePad_1x01_SMD_0.7x2mm
- D18, D23, D3, D8, J14, J15, J16, J17, J18, J19, J24, J25: footprint 0_footprint_Library:SolderWirePad_1x01_SMD_0.5x0.5mm -> 0_footprint_Library:SolderWirePad_1x01_SMD_0.5x2mm_1
- J10: renamed from J9; footprint 0_footprint_Library:SolderWirePad_1x01_SMD_0.5x0.5mm -> 0_footprint_Library:SolderWirePad_1x01_SMD_0.7x2mm
- J21: renamed from J20; footprint 0_footprint_Library:SolderWirePad_1x01_SMD_0.5x0.5mm -> 0_footprint_Library:SolderWirePad_1x01_SMD_0.5x2mm_1
- J22: renamed from J21; footprint 0_footprint_Library:SolderWirePad_1x01_SMD_0.5x0.5mm -> 0_footprint_Library:SolderWirePad_1x01_SMD_0.5x2mm_1
- J23: renamed from J22; footprint 0_footprint_Library:SolderWirePad_1x01_SMD_0.5x0.5mm -> 0_footprint_Library:SolderWirePad_1x01_SMD_0.5x2mm_1
- J8: renamed from J7; footprint 0_footprint_Library:SolderWirePad_1x01_SMD_0.5x0.5mm -> 0_footprint_Library:SolderWirePad_1x01_SMD_0.7x2mm
- J9: renamed from J8; footprint 0_footprint_Library:SolderWirePad_1x01_SMD_0.5x0.5mm -> 0_footprint_Library:SolderWirePad_1x01_SMD_0.7x2mm
- moved J25 6.25 mm to (8.30, 25.5)
- moved D25 6.17 mm to (27.2, 38.0)
- moved J12 5.86 mm to (9.10, 25.5)
- moved D12 5.86 mm to (26.3, 38.0)
- moved J1 5.57 mm to (26.7, 25.5)
- moved D24 5.55 mm to (25.4, 38.0)
- moved J24 5.47 mm to (9.90, 25.5)
- moved D11 5.25 mm to (24.5, 38.0)
- moved J14 5.19 mm to (25.9, 25.5)
- moved J11 5.06 mm to (10.7, 25.5)
- moved D23 4.90 mm to (23.7, 38.0)
- moved J2 4.82 mm to (25.1, 25.5)
- moved D10 4.53 mm to (22.9, 38.0)
- moved J15 4.46 mm to (24.3, 25.5)
- moved D1 4.30 mm to (7.30, 38.0)
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- renumbered J13 to J99
Connections:
- J10 pad 1: Net-(J9-Pin_1) -> Net-(J10-Pin_1)
- J21 pad 1: Net-(J13-P20) -> Net-(J21-Pin_1)
- J22 pad 1: Net-(J13-P21) -> Net-(J22-Pin_1)
- J23 pad 1: Net-(J13-P22) -> Net-(J23-Pin_1)
- J26 pad 13: unconnected-(J26-Pad13) -> Net-(D13-Pin_1)
- J8 pad 1: Net-(J7-Pin_1) -> Net-(J8-Pin_1)
- J9 pad 1: Net-(J8-Pin_1) -> Net-(J9-Pin_1)
- J99 pad 13: unconnected-(J13-Pad13) -> Net-(J13-Pin_1)
- J99 pad 20: Net-(J13-P20) -> Net-(J20-Pin_1)
- J99 pad 21: Net-(J13-P21) -> Net-(J21-Pin_1)
- J99 pad 22: Net-(J13-P22) -> Net-(J22-Pin_1)
- J99 pad 23: Net-(J13-P23) -> Net-(J23-Pin_1)
Routing:
- net Net-(J13-Pin_1): track 0.00 -> 27.4 mm
- net Net-(J22-Pin_1): track 0.00 -> 27.3 mm
- net Net-(D13-Pin_1): track 0.00 -> 27.3 mm
- net Net-(J23-Pin_1): track 0.00 -> 27.1 mm
- net Net-(J21-Pin_1): track 0.00 -> 21.4 mm
- net Net-(J20-Pin_1): track 0.00 -> 21.0 mm
- net Net-(J13-P20): track 20.5 -> 0.00 mm, vias 1 -> 0
- net Net-(J13-P21): track 20.3 -> 0.00 mm, vias 1 -> 0
- net Net-(J13-P23): track 17.9 -> 0.00 mm, vias 1 -> 0
- net Net-(D21-Pin_1): track 16.9 -> 34.5 mm, vias 1 -> 0
- net Net-(J13-P22): track 17.4 -> 0.00 mm, vias 1 -> 0
- net Net-(D9-Pin_1): track 18.3 -> 34.9 mm, vias 1 -> 0
- net Net-(D22-Pin_1): track 17.5 -> 32.7 mm, vias 1 -> 0
- net Net-(D10-Pin_1): track 18.9 -> 33.1 mm, vias 1 -> 0
- net Net-(D23-Pin_1): track 18.0 -> 31.6 mm, vias 1 -> 0
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Other:
- outline, holes or cut-outs redrawn
- board text added: "G"
