File: micro-d-tes-aaray - KICAD/micro-d-tes-aaray.kicad_sch (KiCad schematic)
At the start: 56 parts, among them J1 Conn_01x01_Socket, J10 Conn_01x01_Socket, J11 Conn_01x01_Socket, J12 Conn_01x01_Socket, J13 Conn_01x01_Socket, J14 Conn_01x01_Socket, J15 Conn_01x01_Socket, J16 Conn_01x01_Socket, J17 Conn_01x01_Socket, J18 Conn_01x01_Socket, J19 Conn_01x01_Socket, J2 Conn_01x01_Socket, J20 Conn_01x01_Socket, J21 Conn_01x01_Socket, J22 Conn_01x01_Socket, J23 Conn_01x01_Socket, J24 Conn_01x01_Socket, J25 Conn_01x01_Socket, J26 DB25_Plug, J3 Conn_01x01_Socket, J4 Conn_01x01_Socket, J5 Conn_01x01_Socket, J6 Conn_01x01_Socket, J7 Conn_01x01_Socket, J8 Conn_01x01_Socket, J9 Conn_01x01_Socket, J99 DB25_Plug

Commit message: update
Parts:
- D1, D10, D11, D12, D14, D15, D16, D17, D19, D2, D20, D21, D22, D24, D25, D4, D5, D6, D7, D9, J1, J10, J11, J12, J13, J2, J3, J4, J5, J6, J7, J8, J9: footprint 0_footprint_Library:SolderWirePad_1x01_SMD_0.7x2mm -> 0_footprint_Library:SolderWirePad_1x01_SMD_0.258x2mm
